File: Kicad/Rev A/SHHMduino.kicad_pcb (KiCad board)
At the start: 2 copper layers, 59.9 x 94 mm, 84 parts, among them IC1 ATMEGA328P, IC2 CH340G, P1 ICSP, P2 3V3 GPIO, P3 5V GPIO, P4 Power, P6 Analog, P7 USB, P8 ESP-01, P9 ESP GPIO, Q1 BSS138, Q10 BSS138, Q11 BSS138, Q12 BSS138, Q13 BSS138, Q14 BSS138, Q15 BSS138, Q16 BSS138, Q2 BSS138, Q3 BSS138, Q4 BSS138, Q5 BSS138, Q6 BSS138, Q7 BSS138, Q8 BSS138, Q9 BSS138, SW1 Reset, SW2 ESP Reset, U1 AMS1117, Y1 16mhz, Y2 12mhz

Commit message: Rev A
Rev A silkscreen added
Other:
- board text added: "Rev A"
Changed lines of the file:
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@@
     (area 117.147799 53.264999 181.7192 151.1122)
     (thickness 1.6)
-    (drawings 66)
+    (drawings 68)
     (tracks 1104)
     (zones 0)
@@
       (plotvalue true)
       (plotinvisibletext false)
-      (padsonsilk true)
+      (padsonsilk false)
       (subtractmaskfromsilk false)
       (outputformat 1)
@@
       (xy 4.847166 -4.555643)) (layer F.SilkS) (width 0.01))
   )
+  (gr_text "Rev A" (at 172.974 55.245 180) (layer B.SilkS)
+    (effects (font (size 1.5 1.5) (thickness 0.3)) (justify mirror))
+  )
+  (gr_text "Rev A" (at 175.514 138.176 90) (layer F.SilkS)
+    (effects (font (size 1.5 1.5) (thickness 0.3)))
+  )
   (gr_text "All project files can be found at\n\nhttps://github.com/thermalhound/Shhmduino\n\nThis is an experimental project and must\nbe used at your own risk!" (at 155.829 128.778 180) (layer B.SilkS)
